File: tipi.kicad_pcb (KiCad board)
At the start: 2 copper layers, 100 x 56.5 mm, 32 parts, among them J1 TI32kSideport, Q1 Q_NPN_BCE, T1 TEST_1P, T2 TEST_1P, T3 TEST_1P, T4 TEST_1P, T5 TEST_1P, U1 XC95144XL-TQ100, U2 27C256, U3 74HCT245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

Commit message: Add files via upload
Other:
- board text added: "github.com/lucedoriente/ TI99-4A-internal-TIPI.git"
- board text removed: "github.com/jedimatt42/tipi"
Changed lines of the file:
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@@
 		(layer "Edge.Cuts")
 	)
-	(gr_text "github.com/jedimatt42/tipi"
-		(at 101.4984 152.019 0)
+	(gr_text "github.com/lucedoriente/\nTI99-4A-internal-TIPI.git"
+		(at 104.4956 138.3792 0)
 		(layer "F.SilkS")
 		(effects
 			(font
-				(size 1.5 1.5)
+				(size 1.4 1.4)
 				(thickness 0.3)
 			)
@@
 	)
 	(gr_text "TIPI rev1 for TI/99-24A\noriginal ElectricLab & Jedimatt42\nlayout Alessio Iodice"
-		(at 101.8032 136.3472 0)
+		(at 104.1146 132.8166 0)
 		(layer "F.SilkS")
 		(effects
 			(font
-				(size 1.5 1.5)
+				(size 1.4 1.4)
 				(thickness 0.3)
 			)
